File: kicad/rusmed_eps/rusmed_eps.kicad_pcb (KiCad board)
At the start: 2 copper layers, 84.5 x 57 mm, 14 parts, among them J1 Bornera, J2 Bornera, J3 Bornera, J4 Conn_01x04_Pin

Commit message: [Update]
Parts:
- removed J4: Conn_01x04_Pin, Connector_PinHeader_2.54mm:PinHeader_1x04_P2.54mm_Vertical
- added C1: C, Capacitor_THT:C_Radial_D10.0mm_H16.0mm_P5.00mm, F.Cu at (106.5, 103.5)
- added J5: Molex Microfit 3.0, Connector_Molex:Molex_Micro-Fit_3.0_43045-0612_2x03_P3.00mm_Vertical, F.Cu at (169.0, 99.0)
- added REF**: hw_0468, rusmed:hw_0468, F.Cu at (139.5, 89.0)
- moved D1 35.0 mm to (111.2, 69.5)
- moved REF** 27.9 mm to (135.0, 110.5)
- moved R1 23.4 mm to (102.0, 75.5), turned to 0 degrees
- moved R2 9.40 mm to (149.0, 66.0), turned to 180 degrees
- moved J2 5.66 mm to (173.2, 91.5), turned to 90 degrees
- moved J1 4.53 mm to (103.5, 86.5), turned to -90 degrees
- moved J3 1.64 mm to (173.3, 79.5)
- moved D2 1.12 mm to (130.7, 66.0)
Connections:
- J2 pad 2: +12V -> +5V
Routing:
- net +5V: track 0.00 -> 193.9 mm
- net GND: track 160.0 -> 0.00 mm
- net +12V: track 86.8 -> 117.4 mm
- net Net-(D2-A): track 0.00 -> 5.58 mm
- net Net-(D1-A): track 11.0 -> 6.66 mm
Other:
- board text added: "RUSMED - EPS"
- board text added: "v0.1 - PAI Project"

Commit message: [Update] test
Parts:
- removed the REF** at (139.5, 89.0)
- added U1: U, rusmed:hw_0468, F.Cu at (139.2, 88.2)
- moved R1 2.24 mm to (100.3, 77.0)
- moved D1 1.84 mm to (112.8, 70.5), turned to 180 degrees
- moved D2 1.00 mm to (130.7, 67.0)
- moved R2 1.00 mm to (149.0, 67.0)
- renumbered REF** to M1, REF** to M2, REF** to M3, REF** to M4
Routing:
- net +5V: track 193.9 -> 210.0 mm
- net +12V: track 117.4 -> 120.1 mm
Other:
- board text added: "12V"
- board text added: "Buck converter 5V@25W"
- board text added: "Main supply Bus"
