File: kicad/rusmed_eps/rusmed_eps.kicad_sch (KiCad schematic)
At the start: 8 parts, among them J1 Bornera, J2 Bornera, J3 Bornera, J4 Conn_01x04_Pin

Commit message: [Update]
Parts:
- removed J4: Conn_01x04_Pin, Connector_PinHeader_2.54mm:PinHeader_1x04_P2.54mm_Vertical, symbol Connector:Conn_01x04_Pin
- added C1: C, Capacitor_THT:C_Radial_D10.0mm_H16.0mm_P5.00mm, symbol Device:C
- added J5: Molex Microfit 3.0, Connector_Molex:Molex_Micro-Fit_3.0_43045-0612_2x03_P3.00mm_Vertical, symbol Connector:Conn_01x06_Socket
Connections:
- net +12V: now also C1.1, J5.1 (Pin_1), J5.2 (Pin_2); no longer J2.2 (Pin_2)
- net +5V: now also J2.2 (Pin_2), J5.4 (Pin_4), J5.5 (Pin_5)
- net GND: now also C1.2, J5.3 (Pin_3), J5.6 (Pin_6)
Other:
- moved on the sheet: D1, D2, J1, J2, J3, R1, R2

Commit message: [Update] test
Parts:
- added U1: U, rusmed:hw_0468, symbol rusmed:HW_648
Connections:
- net +12V: now also U1.1 (Vin)
- net +5V: now also U1.3 (Vout)
- net GND: now also U1.2 (GND)

Commit message: [New] Docker compose information
Other:
- note added: "Buck 5V"
- note added: "Led indicadores de alimentacion"
- company: (none) -> RUSMED
- title: (none) -> EPS - Sistema de potencia 
- moved on the sheet: C1, D1, D2, J1, J2, J3, J5, R1, R2, U1
